File: synth-audiocontrols/synth-audiocontrols.kicad_sch (KiCad schematic)
At the start: 13 parts, among them J2 Connector, SW21 Octave_Up, SW25 Octave_Down

Commit message: mounting holes
Parts:
- added H1, H2, H3, H4: MountingHole, MountingHole:MountingHole_3.2mm_M3, symbol Mechanical:MountingHole
