File: synth-audiocontrols/synth-audiocontrols.kicad_pcb (KiCad board)
At the start: 2 copper layers, 95.4 x 57.3 mm, 13 parts, among them J2 Connector, SW21 Octave_Up, SW25 Octave_Down

Commit message: mounting holes
Parts:
- added H1: MountingHole, MountingHole:MountingHole_3.2mm_M3, F.Cu at (114.0, 58.0)
- added H2: MountingHole, MountingHole:MountingHole_3.2mm_M3, F.Cu at (201.0, 58.0)
- added H3: MountingHole, MountingHole:MountingHole_3.2mm_M3, F.Cu at (114.0, 119.5)
- added H4: MountingHole, MountingHole:MountingHole_3.2mm_M3, F.Cu at (201.0, 119.5)
Other:
- board size 95.4 x 57.3 mm -> 95.5 x 68.8 mm

Commit message: Manufacturing changes & Gerber files
Routing:
- net /OCTAVE_UP: track 52.1 -> 61.0 mm
- net /ADC_DIST: track 65.4 -> 71.1 mm, vias 0 -> 5
- net /ADC_MIDS: track 51.0 -> 55.9 mm, vias 0 -> 1
- net /OCTAVE_DOWN: track 33.1 -> 36.7 mm, vias 0 -> 1
- net /ADC_BASS: track 63.6 -> 65.8 mm, vias 0 -> 8
- net /ADC_DELAY: track 36.8 -> 39.0 mm
- net /VOLUME: track 46.5 -> 46.6 mm, vias 0 -> 3
- net /ADC_TREBLE: track 44.2 -> 44.1 mm, vias 0 -> 1
- net /ADC_CHOR: track 42.2 -> 42.3 mm, vias 0 -> 2
- net /ADC_REVERB: vias 0 -> 2
- net GND: vias 31 -> 40
Other:
- board text added: "Team PEAK - ECEN1400 100-1"
