File: synth-loopmatrix/synth-loopmatrix.kicad_sch (KiCad schematic)
At the start: 20 parts, among them J1 Connector, SW1 SaveChord, SW10 Loop1, SW11 Loop2, SW12 Loop3, SW13 Loop4, SW14 Loop5, SW2 PrevChord, SW3 NextChord, SW4 BeginChord, SW5 EndChord, SW6 StartLoop, SW7 SaveLoop, SW8 PauseLoop, SW9 KeyLock

Commit message: mounting holes
Parts:
- added H1, H2, H3, H4: MountingHole, MountingHole:MountingHole_3.2mm_M3, symbol Mechanical:MountingHole
