File: synth-loopmatrix/synth-loopmatrix.kicad_pcb (KiCad board)
At the start: 2 copper layers, 95 x 69 mm, 20 parts, among them J1 Connector, SW1 SaveChord, SW10 Loop1, SW11 Loop2, SW12 Loop3, SW13 Loop4, SW14 Loop5, SW2 PrevChord, SW3 NextChord, SW4 BeginChord, SW5 EndChord, SW6 StartLoop, SW7 SaveLoop, SW8 PauseLoop, SW9 KeyLock

Commit message: mounting holes
Parts:
- added H1: MountingHole, MountingHole:MountingHole_3.2mm_M3, F.Cu at (89.0, 48.0)
- added H2: MountingHole, MountingHole:MountingHole_3.2mm_M3, F.Cu at (177.0, 48.0)
- added H3: MountingHole, MountingHole:MountingHole_3.2mm_M3, F.Cu at (89.0, 121.0)
- added H4: MountingHole, MountingHole:MountingHole_3.2mm_M3, F.Cu at (177.0, 121.0)
Other:
- board size 95 x 69 mm -> 95 x 80 mm

Commit message: implement design suggestions from TA
Parts:
- moved R2 1.10 mm to (102.8, 108.0), turned to 0 degrees
Routing:
- net /COL1: track 63.1 -> 78.8 mm
- net /ROW3: track 95.0 -> 108.3 mm
- net /COL2: track 66.0 -> 75.2 mm
- net /COL5: track 125.5 -> 133.8 mm
- net /COL3: track 80.7 -> 89.0 mm
- net /LOCK_LED: track 141.1 -> 136.5 mm
- net /COL4: track 103.1 -> 107.0 mm
- net /ROW2: track 116.6 -> 119.7 mm
- net /ROW1: track 136.2 -> 137.3 mm
- net GND: vias 19 -> 18

Commit message: Manufacturing changes & Gerber files
Routing:
- net /ROW3: track 108.3 -> 109.7 mm
- net /ROW2: track 119.7 -> 120.3 mm
- net /ROW1: track 137.3 -> 138.0 mm
Other:
- board text added: "Team PEAK - ECEN1400 100-1"
Changed lines of the file:
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@@
 			(outputformat 1)
 			(mirror no)
-			(drillshape 1)
+			(drillshape 0)
 			(scaleselection 1)
-			(outputdirectory "")
+			(outputdirectory "Gerbers/")
 		)
 	)
@@
 		(layer "Edge.Cuts")
 	)
+	(gr_text "Team PEAK - ECEN1400 100-1"
+		(at 155.3 121 0)
+		(layer "F.SilkS")
+		(effects
+			(font
+				(size 1.5 1.5)
+				(thickness 0.3)
+				(bold yes)
+			)
+		)
+	)
+	(dimension
+		(type orthogonal)
+		(layer "F.Fab")
+		(pts
+			(xy 85.5 44.5) (xy 85.5 124.5)
+		)
+		(height -5.5)
+		(orientation 1)
+		(format
+			(prefix "")
+			(suffix "")
+			(units 3)
+			(units_format 0)
+			(precision 4)
+			(suppress_zeroes yes)
+		)
+		(style
+			(thickness 0.1)
+			(arrow_length 1.27)
+			(text_position_mode 0)
+			(arrow_direction outward)
+			(extension_height 0.58642)
+			(extension_offset 0.5)
+			(keep_text_aligned yes)
+		)
+		(gr_text "80"
+			(at 78.85 84.5 90)
+			(layer "F.Fab")
+			(effects
+				(font
+					(size 1 1)
+					(thickness 0.15)
+				)
+			)
+		)
+	)
+	(dimension
+		(type orthogonal)
+		(layer "F.Fab")
+		(pts
+			(xy 180.5 44.5) (xy 85.5 44.5)
+		)
+		(height -4.5)
+		(orientation 0)
+		(format
+			(prefix "")
+			(suffix "")
+			(units 3)
+			(units_format 0)
+			(precision 4)
+			(suppress_zeroes yes)
+		)
+		(style
+			(thickness 0.1)
+			(arrow_length 1.27)
+			(text_position_mode 0)
+			(arrow_direction outward)
+			(extension_height 0.58642)
+			(extension_offset 0.5)
+			(keep_text_aligned yes)
+		)
+		(gr_text "95"
+			(at 133 38.85 0)
+			(layer "F.Fab")
+			(effects
+				(font
+					(size 1 1)
+					(thickness 0.15)
+				)
+			)
+		)
+	)
 	(via
 		(at 101 105)
@@
 	)
 	(via
-		(at 143.5 115)
+		(at 142.5 115)
 		(size 0.7)
 		(drill 0.4)
@@
 	)
 	(via
-		(at 124.5 115)
+		(at 123.6 115)
 		(size 0.7)
 		(drill 0.4)
@@
 	)
 	(via
-		(at 105.7 90.5)
+		(at 105.2 90.4)
 		(size 0.7)
 		(drill 0.4)
@@
 	)
 	(segment
+		(start 172.72 53.6)
+		(end 173.54 54.42)
+		(width 0.5)
+		(layer "F.Cu")
+		(net "/ROW1")
+	)
+	(segment
 		(start 103.8875 108.6125)
 		(end 101.54 110.96)
@@
 	)
 	(segment
+		(start 98.36 53.6)
+		(end 172.72 53.6)
+		(width 0.5)
+		(layer "F.Cu")
+		(net "/ROW1")
+	)
+	(segment
 		(start 99.42 54.42)
 		(end 97.54 54.42)
@@
 	(segment
 		(start 97.54 54.42)
-		(end 173.54 54.42)
+		(end 98.36 53.6)
 		(width 0.5)
 		(layer "F.Cu")
@@
 	)
 	(segment
-		(start 97.54 109.88)
-		(end 97.54 108.24)
+		(start 97.54 108.24)
+		(end 87.7 98.4)
 		(width 0.5)
 		(layer "F.Cu")
@@
 	)
 	(segment
-		(start 87.7 93.4)
-		(end 88.68 92.42)
+		(start 173.54 92.42)
+		(end 172.72 91.6)
 		(width 0.5)
 		(layer "F.Cu")
@@
 	)
 	(segment
-		(start 97.54 108.24)
-		(end 87.7 98.4)
+		(start 97.54 109.88)
+		(end 97.54 108.24)
 		(width 0.5)
 		(layer "F.Cu")
@@
 	)
 	(segment
-		(start 87.7 98.4)
-		(end 87.7 93.4)
+		(start 96.72 91.6)
+		(end 97.54 92.42)
+		(width 0.5)
+		(layer "F.Cu")
+		(net "/ROW3")
+	)
+	(segment
+		(start 172.72 91.6)
+		(end 98.36 91.6)
 		(width 0.5)
 		(layer "F.Cu")
@@
 	)
 	(segment
-		(start 88.68 92.42)
+		(start 98.36 91.6)
 		(end 97.54 92.42)
 		(width 0.5)
@@
 	)
 	(segment
-		(start 173.54 92.42)
-		(end 97.54 92.42)
+		(start 87.7 98.4)
+		(end 87.7 93.4)
+		(width 0.5)
+		(layer "F.Cu")
+		(net "/ROW3")
+	)
+	(segment
+		(start 89.5 91.6)
+		(end 96.72 91.6)
+		(width 0.5)
+		(layer "F.Cu")
+		(net "/ROW3")
+	)
+	(segment
+		(start 87.7 93.4)
+		(end 89.5 91.6)
 		(width 0.5)
 		(layer "F.Cu")
@@
 	)
 	(segment
+		(start 98.36 72.6)
+		(end 97.54 73.42)
+		(width 0.5)
+		(layer "F.Cu")
+		(net "/ROW2")
+	)
+	(segment
 		(start 102.6 99.2)
 		(end 99 102.8)
@@
 	)
 	(segment
+		(start 172.72 72.6)
+		(end 98.36 72.6)
+		(width 0.5)
+		(layer "F.Cu")
+		(net "/ROW2")
+	)
+	(segment
 		(start 101.1 75.8)
 		(end 99.9 75.8)
@@
 	(segment
 		(start 173.54 73.42)
-		(end 97.54 73.42)
+		(end 172.72 72.6)
 		(width 0.5)
 		(layer "F.Cu")
@@
 	)
 	(segment
+		(start 91.19 94.96)
+		(end 87.7 91.47)
+		(width 0.5)
+		(layer "B.Cu")
+		(net "/COL1")
+	)
+	(segment
 		(start 104 111.04)
 		(end 104 110.035534)
@@
 	)
 	(segment
-		(start 87.7 96.2)
-		(end 87.7 77.9)
-		(width 0.5)
-		(layer "B.Cu")
-		(net "/COL1")
-	)
-	(segment
 		(start 87.7 71.8)
 		(end 87.7 58.7)
@@
 		(width 0.5)
 		(layer "B.Cu")
+		(net "/COL1")
+	)
+	(segment
+		(start 87.7 91.47)
+		(end 87.7 77.9)
+		(width 0.5)
+		(layer "B.Cu")
